File: SRC/MCU_ATMEGA328P-M.kicad_sch (KiCad schematic)
At the start: 33 parts, among them SW301 SW_AUTO, SW302 SW_TIME, SW303 SW_DAY, SW304 SW_RST, SW305 SW_HOUR, SW306 SW_MIN, SW307 SW_PROG, U301 ATmega328P-M, U302 SX1M32.768KM10F30TN, Y301 16MHz

Commit message: Added debug testpoints.
Parts:
- added TP301: TP_MOSI, TestPoint:TestPoint_Pad_D1.5mm, symbol Connector:TestPoint
- added TP302: TP_VCC, TestPoint:TestPoint_Pad_D1.5mm, symbol Connector:TestPoint
- added TP303: TP_MISO, TestPoint:TestPoint_Pad_D1.5mm, symbol Connector:TestPoint
- added TP304: TP_RST, TestPoint:TestPoint_Pad_D1.5mm, symbol Connector:TestPoint
- added TP305: TP_SCK, TestPoint:TestPoint_Pad_D1.5mm, symbol Connector:TestPoint
- added TP306: TP_GND, TestPoint:TestPoint_Pad_D1.5mm, symbol Connector:TestPoint
Connections:
- net +3V3: now also TP302.1
- net GND: now also TP306.1
- net NRST: now also TP304.1
- net PB4: now also TP303.1
- net PB5: now also TP305.1
- net BTN_AUTO renamed PD6
- net BTN_DAY renamed PB0
- net BTN_HOUR renamed PB2
- net BTN_MIN renamed PB3
- net PB3: now also TP301.1
- net BTN_PROG renamed PB1
- net BTN_TIME renamed PD7
Other:
- note added: "ATMEGA328P"
- note added: "DEBUG TESTPOINTS"
