File: SRC/MODULE_LCD1602_4BIT.kicad_sch (KiCad schematic)
At the start: 9 parts, among them Q401 MMBT3904

Commit message: Added debug testpoints.
Parts:
- renumbered R404 to R401
Changed lines of the file:
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@@
   (symbol (lib_id "Device:R_Small") (at 72.39 97.79 0) (mirror y) (unit 1)
     (in_bom yes) (on_board yes) (dnp no) (fields_autoplaced)
-    (property "Reference" "R404" (at 74.93 97.155 0)
+    (property "Reference" "R401" (at 74.93 97.155 0)
       (effects (font (size 1.27 1.27)) (justify right))
     )
@@
       (project "Digital_Timer_Switch"
         (path "/98b51aac-404f-4a0d-b314-bd3823594ee3/ef1ab763-c83c-4112-b155-97ec3ec1921c"
-          (reference "R404") (unit 1)
+          (reference "R401") (unit 1)
         )
       )
